Commit message: Allowing multirobot

File: models/iris/iris.sdf.xacro (robot description, xacro)
@@ -7,6 +7,7 @@
   <xacro:arg name='camera_udp_port' default='5600' />
   <xacro:arg name='rotors_description_dir' default='.'/>
+  <xacro:arg name='vehicle_name' default='iris'/>
   <model name='iris'>
-    <link name='base_link'>
+    <link name='$(arg vehicle_name)_base_link'>
       <pose frame=''>0 0 0 0 -0 0</pose>
       <inertial>
@@ -22,5 +23,5 @@
         </inertia>
       </inertial>
-      <collision name='base_link_inertia_collision'>
+      <collision name='$(arg vehicle_name)_base_link_inertia_collision'>
         <pose frame=''>0 0 0 0 -0 0</pose>
         <geometry>
@@ -41,5 +42,5 @@
         </surface>
       </collision>
-      <visual name='base_link_inertia_visual'>
+      <visual name='$(arg vehicle_name)_base_link_inertia_visual'>
         <pose frame=''>0 0 0 0 -0 0</pose>
         <geometry>
@@ -60,5 +61,5 @@
       <self_collide>0</self_collide>
     </link>
-    <link name='/imu_link'>
+    <link name='$(arg vehicle_name)_imu_link'>
       <pose frame=''>0 0 0 0 -0 0</pose>
       <inertial>
@@ -75,7 +76,7 @@
       </inertial>
     </link>
-    <joint name='/imu_joint' type='revolute'>
-      <child>/imu_link</child>
-      <parent>base_link</parent>
+    <joint name='imu_joint' type='revolute'>
+      <child>$(arg vehicle_name)_imu_link</child>
+      <parent>$(arg vehicle_name)_base_link</parent>
       <axis>
         <xyz>1 0 0</xyz>
@@ -93,5 +94,5 @@
       </axis>
     </joint>
-    <link name='rotor_0'>
+    <link name='$(arg vehicle_name)_rotor_0'>
       <pose frame=''>0.13 -0.22 0.023 0 -0 0</pose>
       <inertial>
@@ -107,5 +108,5 @@
         </inertia>
       </inertial>
-      <collision name='rotor_0_collision'>
+      <collision name='$(arg vehicle_name)_rotor_0_collision'>
         <pose frame=''>0 0 0 0 -0 0</pose>
         <geometry>
@@ -124,5 +125,5 @@
         </surface>
       </collision>
-      <visual name='rotor_0_visual'>
+      <visual name='$(arg vehicle_name)_rotor_0_visual'>
         <pose frame=''>0 0 0 0 -0 0</pose>
         <geometry>
@@ -143,7 +144,7 @@
       <self_collide>0</self_collide>
     </link>
-    <joint name='rotor_0_joint' type='revolute'>
-      <child>rotor_0</child>
-      <parent>base_link</parent>
+    <joint name='$(arg vehicle_name)_rotor_0_joint' type='revolute'>
+      <child>$(arg vehicle_name)_rotor_0</child>
+      <parent>$(arg vehicle_name)_base_link</parent>
       <axis>
         <xyz>0 0 1</xyz>
@@ -159,5 +160,5 @@
       </axis>
     </joint>
-    <link name='rotor_1'>
+    <link name='$(arg vehicle_name)_rotor_1'>
       <pose frame=''>-0.13 0.2 0.023 0 -0 0</pose>
       <inertial>
@@ -173,5 +174,5 @@
         </inertia>
       </inertial>
-      <collision name='rotor_1_collision'>
+      <collision name='$(arg vehicle_name)_rotor_1_collision'>
         <pose frame=''>0 0 0 0 -0 0</pose>
         <geometry>
@@ -190,5 +191,5 @@
         </surface>
       </collision>
-      <visual name='rotor_1_visual'>
+      <visual name='$(arg vehicle_name)_rotor_1_visual'>
         <pose frame=''>0 0 0 0 -0 0</pose>
         <geometry>
@@ -209,7 +210,7 @@
       <self_collide>0</self_collide>
     </link>
-    <joint name='rotor_1_joint' type='revolute'>
-      <child>rotor_1</child>
-      <parent>base_link</parent>
+    <joint name='$(arg vehicle_name)_rotor_1_joint' type='revolute'>
+      <child>$(arg vehicle_name)_rotor_1</child>
+      <parent>$(arg vehicle_name)_base_link</parent>
       <axis>
         <xyz>0 0 1</xyz>
@@ -225,5 +226,5 @@
       </axis>
     </joint>
-    <link name='rotor_2'>
+    <link name='$(arg vehicle_name)_rotor_2'>
       <pose frame=''>0.13 0.22 0.023 0 -0 0</pose>
       <inertial>
@@ -239,5 +240,5 @@
         </inertia>
       </inertial>
-      <collision name='rotor_2_collision'>
+      <collision name='$(arg vehicle_name)_rotor_2_collision'>
         <pose frame=''>0 0 0 0 -0 0</pose>
         <geometry>
@@ -256,5 +257,5 @@
         </surface>
       </collision>
-      <visual name='rotor_2_visual'>
+      <visual name='$(arg vehicle_name)_rotor_2_visual'>
         <pose frame=''>0 0 0 0 -0 0</pose>
         <geometry>
@@ -275,7 +276,7 @@
       <self_collide>0</self_collide>
     </link>
-    <joint name='rotor_2_joint' type='revolute'>
-      <child>rotor_2</child>
-      <parent>base_link</parent>
+    <joint name='$(arg vehicle_name)_rotor_2_joint' type='revolute'>
+      <child>$(arg vehicle_name)_rotor_2</child>
+      <parent>$(arg vehicle_name)_base_link</parent>
       <axis>
         <xyz>0 0 1</xyz>
@@ -291,5 +292,5 @@
       </axis>
     </joint>
-    <link name='rotor_3'>
+    <link name='$(arg vehicle_name)_rotor_3'>
       <pose frame=''>-0.13 -0.2 0.023 0 -0 0</pose>
       <inertial>
@@ -305,5 +306,5 @@
         </inertia>
       </inertial>
-      <collision name='rotor_3_collision'>
+      <collision name='$(arg vehicle_name)_rotor_3_collision'>
         <pose frame=''>0 0 0 0 -0 0</pose>
         <geometry>
@@ -322,5 +323,5 @@
         </surface>
       </collision>
-      <visual name='rotor_3_visual'>
+      <visual name='$(arg vehicle_name)_rotor_3_visual'>
         <pose frame=''>0 0 0 0 -0 0</pose>
         <geometry>
@@ -341,7 +342,7 @@
       <self_collide>0</self_collide>
     </link>
-    <joint name='rotor_3_joint' type='revolute'>
-      <child>rotor_3</child>
-      <parent>base_link</parent>
+    <joint name='$(arg vehicle_name)_rotor_3_joint' type='revolute'>
+      <child>$(arg vehicle_name)_rotor_3</child>
+      <parent>$(arg vehicle_name)_base_link</parent>
       <axis>
         <xyz>0 0 1</xyz>
@@ -359,11 +360,11 @@
     <plugin name='rosbag' filename='libgazebo_multirotor_base_plugin.so'>
       <robotNamespace/>
-      <linkName>base_link</linkName>
+      <linkName>$(arg vehicle_name)_base_link</linkName>
       <rotorVelocitySlowdownSim>10</rotorVelocitySlowdownSim>
     </plugin>
     <plugin name='front_right_motor_model' filename='libgazebo_motor_model.so'>
       <robotNamespace/>
-      <jointName>rotor_0_joint</jointName>
-      <linkName>rotor_0</linkName>
+      <jointName>$(arg vehicle_name)_rotor_0_joint</jointName>
+      <linkName>$(arg vehicle_name)_rotor_0</linkName>
       <turningDirection>ccw</turningDirection>
       <timeConstantUp>0.0125</timeConstantUp>
@@ -381,6 +382,6 @@
     <plugin name='back_left_motor_model' filename='libgazebo_motor_model.so'>
       <robotNamespace/>
-      <jointName>rotor_1_joint</jointName>
-      <linkName>rotor_1</linkName>
+      <jointName>$(arg vehicle_name)_rotor_1_joint</jointName>
+      <linkName>$(arg vehicle_name)_rotor_1</linkName>
       <turningDirection>ccw</turningDirection>
       <timeConstantUp>0.0125</timeConstantUp>
@@ -398,6 +399,6 @@
     <plugin name='front_left_motor_model' filename='libgazebo_motor_model.so'>
       <robotNamespace/>
-      <jointName>rotor_2_joint</jointName>
-      <linkName>rotor_2</linkName>
+      <jointName>$(arg vehicle_name)_rotor_2_joint</jointName>
+      <linkName>$(arg vehicle_name)_rotor_2</linkName>
       <turningDirection>cw</turningDirection>
       <timeConstantUp>0.0125</timeConstantUp>
@@ -415,6 +416,6 @@
     <plugin name='back_right_motor_model' filename='libgazebo_motor_model.so'>
       <robotNamespace/>
-      <jointName>rotor_3_joint</jointName>
-      <linkName>rotor_3</linkName>
+      <jointName>$(arg vehicle_name)_rotor_3_joint</jointName>
+      <linkName>$(arg vehicle_name)_rotor_3</linkName>
       <turningDirection>cw</turningDirection>
       <timeConstantUp>0.0125</timeConstantUp>
@@ -566,8 +567,19 @@
       </control_channels>
     </plugin>
+    <plugin name="joint_state_publisher" filename="libgazebo_ros_joint_state_publisher.so">
+      <ros>
+        <namespace>/</namespace>
+        <argument>joint_states:=joint_states</argument>
+      </ros>
+      <joint_name>$(arg vehicle_name)::$(arg vehicle_name)_rotor_0_joint</joint_name>
+      <joint_name>$(arg vehicle_name)::$(arg vehicle_name)_rotor_1_joint</joint_name>
+      <joint_name>$(arg vehicle_name)::$(arg vehicle_name)_rotor_2_joint</joint_name>
+      <joint_name>$(arg vehicle_name)::$(arg vehicle_name)_rotor_3_joint</joint_name>
+      <update_rate>100</update_rate>
+    </plugin>
     <static>0</static>
     <plugin name='rotors_gazebo_imu_plugin' filename='libgazebo_imu_plugin.so'>
       <robotNamespace/>
-      <linkName>/imu_link</linkName>
+      <linkName>$(arg vehicle_name)_imu_link</linkName>
       <imuTopic>/imu</imuTopic>
       <gyroscopeNoiseDensity>0.0003394</gyroscopeNoiseDensity>
@@ -585,5 +597,5 @@
     <joint name="fpv_cam_joint" type="fixed">
       <child>fpv_cam::link</child>
-      <parent>base_link</parent>
+      <parent>$(arg vehicle_name)_base_link</parent>
       <axis>
         <xyz>0 0 1</xyz>

File: models/iris/iris.urdf.xacro (robot description, xacro)
@@ -7,5 +7,6 @@
   <xacro:arg name='camera_udp_port' default='5600' />
   <xacro:arg name='rotors_description_dir' default='.'/>
-    <link name='base_link'>
+  <xacro:arg name='vehicle_name' default='iris'/>
+    <link name='$(arg vehicle_name)_base_link'>
       <pose rpy="0  0  0" xyz="0  0  0"/>
       <inertial>
@@ -14,5 +15,5 @@
         <inertia ixx="0.0347563" ixy="0" ixz="0" iyy="0.0458929" iyz="0" izz="0.0977"/>
       </inertial>
-      <collision name="base_link_inertia_collision">
+      <collision name="$(arg vehicle_name)_base_link_inertia_collision">
         <origin rpy="0  0  0" xyz="0  0  0"/>
         <geometry>
@@ -20,5 +21,5 @@
         </geometry>
       </collision>
-      <visual name="base_link_inertia_visual">
+      <visual name="$(arg vehicle_name)_base_link_inertia_visual">
         <origin rpy="0  0  0" xyz="0  0  0"/>
         <geometry>
@@ -30,5 +31,5 @@
       </visual>
     </link>
-    <gazebo reference="base_link">
+    <gazebo reference="$(arg vehicle_name)_base_link">
       <material>Gazebo/Black</material>
       <gravity>1</gravity>
@@ -36,5 +37,5 @@
       <self_collide>0</self_collide>
     </gazebo>
-    <link name='/imu_link'>
+    <link name='$(arg vehicle_name)_imu_link'>
       <pose rpy="0  0  0" xyz="0  0  0"/>
       <inertial>
@@ -45,11 +46,11 @@
     </link>
     <joint name="imu_joint" type="revolute">
-      <parent link="base_link"/>
-      <child link="/imu_link"/>
+      <parent link="$(arg vehicle_name)_base_link"/>
+      <child link="$(arg vehicle_name)_imu_link"/>
       <origin rpy="0  0  0" xyz="0  0  0"/>
       <axis xyz="1  0  0"/>
       <limit effort="0.0" lower="0.0" upper="0.0" velocity="0.0"/>
     </joint>
-    <link name='rotor_0'>
+    <link name='$(arg vehicle_name)_rotor_0'>
       <pose rpy="0.13 -0.22" xyz="0.023 0 -0 0"/>
       <inertial>
@@ -58,5 +59,5 @@
         <inertia ixx="9.75e-07" ixy="0" ixz="0" iyy="0.000273104" iyz="0" izz="0.000274004"/>
       </inertial>
-      <collision name="rotor_0_collision">
+      <collision name="$(arg vehicle_name)_rotor_0_collision">
         <origin rpy="0  0  0" xyz="0  0  0"/>
         <geometry>
@@ -64,5 +65,5 @@
         </geometry>
       </collision>
-      <visual name="rotor_0_visual">
+      <visual name="$(arg vehicle_name)_rotor_0_visual">
         <origin rpy="0  0  0" xyz="0  0  0"/>
         <geometry>
@@ -74,5 +75,5 @@
       </visual>
     </link>
-    <gazebo reference="rotor_0">
+    <gazebo reference="$(arg vehicle_name)_rotor_0">
       <material>Gazebo/Blue</material>
       <gravity>1</gravity>
@@ -80,12 +81,12 @@
       <self_collide>0</self_collide>
     </gazebo>
-    <joint name="rotor_0_joint" type="revolute">
-      <parent link="base_link"/>
-      <child link="rotor_0"/>
+    <joint name="$(arg vehicle_name)_rotor_0_joint" type="revolute">
+      <parent link="$(arg vehicle_name)_base_link"/>
+      <child link="$(arg vehicle_name)_rotor_0"/>
       <origin rpy="0  0  0" xyz="0.13  -0.22   0.023"/>
       <axis xyz="0  0  1"/>
       <limit effort="0.0" lower="-1e+16" upper="1e+16" velocity="0.0"/>
     </joint>
-    <link name='rotor_1'>
+    <link name='$(arg vehicle_name)_rotor_1'>
       <pose rpy="-0.13 0.2" xyz="0.023 0 -0 0"/>
       <inertial>
@@ -94,5 +95,5 @@
         <inertia ixx="9.75e-07" ixy="0" ixz="0" iyy="0.000273104" iyz="0" izz="0.000274004"/>
       </inertial>
-      <collision name="rotor_1_collision">
+      <collision name="$(arg vehicle_name)_rotor_1_collision">
         <origin rpy="0  0  0" xyz="0  0  0"/>
         <geometry>
@@ -100,5 +101,5 @@
         </geometry>
       </collision>
-      <visual name="rotor_1_visual">
+      <visual name="$(arg vehicle_name)_rotor_1_visual">
         <origin rpy="0  0  0" xyz="0  0  0"/>
         <geometry>
@@ -110,5 +111,5 @@
       </visual>
     </link>
-    <gazebo reference="rotor_1">
+    <gazebo reference="$(arg vehicle_name)_rotor_1">
       <material>Gazebo/Black</material>
       <gravity>1</gravity>
@@ -116,12 +117,12 @@
       <self_collide>0</self_collide>
     </gazebo>
-    <joint name="rotor_1_joint" type="revolute">
-      <parent link="base_link"/>
-      <child link="rotor_1"/>
+    <joint name="$(arg vehicle_name)_rotor_1_joint" type="revolute">
+      <parent link="$(arg vehicle_name)_base_link"/>
+      <child link="$(arg vehicle_name)_rotor_1"/>
       <origin rpy="0  0  0" xyz="-0.13   0.2    0.023"/>
       <axis xyz="0  0  1"/>
       <limit effort="0.0" lower="-1e+16" upper="1e+16" velocity="0.0"/>
     </joint>
-    <link name='rotor_2'>
+    <link name='$(arg vehicle_name)_rotor_2'>
       <pose rpy="0.13 0.2" xyz="0.023 0 -0 0"/>
       <inertial>
@@ -130,5 +131,5 @@
         <inertia ixx="9.75e-07" ixy="0" ixz="0" iyy="0.000273104" iyz="0" izz="0.000274004"/>
       </inertial>
-      <collision name="rotor_2_collision">
+      <collision name="$(arg vehicle_name)_rotor_2_collision">
         <origin rpy="0  0  0" xyz="0  0  0"/>
         <geometry>
@@ -136,5 +137,5 @@
         </geometry>
       </collision>
-      <visual name="rotor_2_visual">
+      <visual name="$(arg vehicle_name)_rotor_2_visual">
         <origin rpy="0  0  0" xyz="0  0  0"/>
         <geometry>
@@ -146,5 +147,5 @@
       </visual>
     </link>
-    <gazebo reference="rotor_2">
+    <gazebo reference="$(arg vehicle_name)_rotor_2">
       <material>Gazebo/Blue</material>
       <gravity>1</gravity>
@@ -152,12 +153,12 @@
       <self_collide>0</self_collide>
     </gazebo>
-    <joint name="rotor_2_joint" type="revolute">
-      <parent link="base_link"/>
-      <child link="rotor_2"/>
+    <joint name="$(arg vehicle_name)_rotor_2_joint" type="revolute">
+      <parent link="$(arg vehicle_name)_base_link"/>
+      <child link="$(arg vehicle_name)_rotor_2"/>
       <origin rpy="0  0  0" xyz="0.13   0.22   0.023"/>
       <axis xyz="0  0  1"/>
       <limit effort="0.0" lower="-1e+16" upper="1e+16" velocity="0.0"/>
     </joint>
-    <link name='rotor_3'>
+    <link name='$(arg vehicle_name)_rotor_3'>
       <pose rpy="-0.13 -0.2" xyz="0.023 0 -0 0"/>
       <inertial>
@@ -166,5 +167,5 @@
         <inertia ixx="9.75e-07" ixy="0" ixz="0" iyy="0.000273104" iyz="0" izz="0.000274004"/>
       </inertial>
-      <collision name="rotor_3_collision">
+      <collision name="$(arg vehicle_name)_rotor_3_collision">
         <origin rpy="0  0  0" xyz="0  0  0"/>
         <geometry>
@@ -172,5 +173,5 @@
         </geometry>
       </collision>
-      <visual name="rotor_3_visual">
+      <visual name="$(arg vehicle_name)_rotor_3_visual">
         <origin rpy="0  0  0" xyz="0  0  0"/>
         <geometry>
@@ -182,5 +183,5 @@
       </visual>
     </link>
-    <gazebo reference="rotor_3">
+    <gazebo reference="$(arg vehicle_name)_rotor_3">
       <material>Gazebo/Black</material>
       <gravity>1</gravity>
@@ -188,7 +189,7 @@
       <self_collide>0</self_collide>
     </gazebo>
-    <joint name="rotor_3_joint" type="revolute">
-      <parent link="base_link"/>
-      <child link="rotor_3"/>
+    <joint name="$(arg vehicle_name)_rotor_3_joint" type="revolute">
+      <parent link="$(arg vehicle_name)_base_link"/>
+      <child link="$(arg vehicle_name)_rotor_3"/>
       <origin rpy="0  0  0" xyz="-0.13  -0.2    0.023"/>
       <axis xyz="0  0  1"/>
@@ -198,11 +199,11 @@
     <plugin name='multirobot_base_plugin' filename='libgazebo_multirotor_base_plugin.so'>
       <robotNamespace/>
-      <linkName>base_link</linkName>
+      <linkName>$(arg vehicle_name)_base_link</linkName>
       <rotorVelocitySlowdownSim>10</rotorVelocitySlowdownSim>
     </plugin>
     <plugin name='front_right_motor_model' filename='libgazebo_motor_model.so'>
       <robotNamespace/>
-      <jointName>rotor_0_joint</jointName>
-      <linkName>rotor_0</linkName>
+      <jointName>$(arg vehicle_name)_rotor_0_joint</jointName>
+      <linkName>$(arg vehicle_name)_rotor_0</linkName>
       <turningDirection>ccw</turningDirection>
       <timeConstantUp>0.0125</timeConstantUp>
@@ -220,6 +221,6 @@
     <plugin name='back_left_motor_model' filename='libgazebo_motor_model.so'>
       <robotNamespace/>
-      <jointName>rotor_1_joint</jointName>
-      <linkName>rotor_1</linkName>
+      <jointName>$(arg vehicle_name)_rotor_1_joint</jointName>
+      <linkName>$(arg vehicle_name)_rotor_1</linkName>
       <turningDirection>ccw</turningDirection>
       <timeConstantUp>0.0125</timeConstantUp>
@@ -237,6 +238,6 @@
     <plugin name='front_left_motor_model' filename='libgazebo_motor_model.so'>
       <robotNamespace/>
-      <jointName>rotor_2_joint</jointName>
-      <linkName>rotor_2</linkName>
+      <jointName>$(arg vehicle_name)_rotor_2_joint</jointName>
+      <linkName>$(arg vehicle_name)_rotor_2</linkName>
       <turningDirection>cw</turningDirection>
       <timeConstantUp>0.0125</timeConstantUp>
@@ -254,6 +255,6 @@
     <plugin name='back_right_motor_model' filename='libgazebo_motor_model.so'>
       <robotNamespace/>
-      <jointName>rotor_3_joint</jointName>
-      <linkName>rotor_3</linkName>
+      <jointName>$(arg vehicle_name)_rotor_3_joint</jointName>
+      <linkName>$(arg vehicle_name)_rotor_3</linkName>
       <turningDirection>cw</turningDirection>
       <timeConstantUp>0.0125</timeConstantUp>
@@ -408,17 +409,17 @@
     <plugin name="joint_state_publisher" filename="libgazebo_ros_joint_state_publisher.so">
       <ros>
-        <namespace>/demo</namespace>
+        <namespace>/</namespace>
         <argument>joint_states:=joint_states</argument>
       </ros>
-      <joint_name>iris_0::imu_link</joint_name>
-      <joint_name>iris_0::rotor_0_joint</joint_name>
-      <joint_name>iris_0::rotor_1_joint</joint_name>
-      <joint_name>iris_0::rotor_2_joint</joint_name>
-      <joint_name>iris_0::rotor_3_joint</joint_name>
+      <joint_name>$(arg vehicle_name)::$(arg vehicle_name)_imu_link</joint_name>
+      <joint_name>$(arg vehicle_name)::$(arg vehicle_name)_rotor_0_joint</joint_name>
+      <joint_name>$(arg vehicle_name)::$(arg vehicle_name)_rotor_1_joint</joint_name>
+      <joint_name>$(arg vehicle_name)::$(arg vehicle_name)_rotor_2_joint</joint_name>
+      <joint_name>$(arg vehicle_name)::$(arg vehicle_name)_rotor_3_joint</joint_name>
       <update_rate>100</update_rate>
     </plugin>
     <plugin name='rotors_gazebo_imu_plugin' filename='libgazebo_imu_plugin.so'>
       <robotNamespace/>
-      <linkName>/imu_link</linkName>
+      <linkName>$(arg vehicle_name)_imu_link</linkName>
       <imuTopic>/imu</imuTopic>
       <gyroscopeNoiseDensity>0.0003394</gyroscopeNoiseDensity>
@@ -437,5 +438,5 @@
     <xacro:fpv_cam/>
     <joint name="fpv_joint" type="fixed">
-      <parent link="base_link"/>
+      <parent link="$(arg vehicle_name)_base_link"/>
       <child link="camera_link"/>
       <origin rpy="0  0  0" xyz="0  0  0"/>
