Commit message: Allowing multirobot

File: models/plane/plane.sdf.xacro (robot description, xacro)
@@ -8,7 +8,8 @@
   <xacro:arg name='camera_control_udp_port' default='14530' />
   <xacro:arg name='rotors_description_dir' default='.'/>
+  <xacro:arg name='vehicle_name' default='iris'/>
   <model name='plane'>
     <pose>0 0 0.246 0 0 0</pose>
-    <link name='base_link'>
+    <link name='$(arg vehicle_name)_base_link'>
       <pose>0 0 0 0 0 0</pose>
       <inertial>
@@ -24,5 +25,5 @@
         </inertia>
       </inertial>
-      <collision name='base_link_collision'>
+      <collision name='$(arg vehicle_name)_base_link_collision'>
         <pose>0 0 -0.07 0 0 0</pose>
         <geometry>
@@ -43,5 +44,5 @@
         </surface>
       </collision>
-      <visual name='base_link_visual'>
+      <visual name='$(arg vehicle_name)_base_link_visual'>
         <pose>0.07 0 -0.08 0 0 0</pose>
         <geometry>
@@ -62,5 +63,5 @@
       <self_collide>0</self_collide>
     </link>
-    <link name='plane/imu_link'>
+    <link name='$(arg vehicle_name)_plane/imu_link'>
       <pose>0 0 0 0 0 0</pose>
       <inertial>
@@ -78,6 +79,6 @@
     </link>
     <joint name='plane/imu_joint' type='revolute'>
-      <child>plane/imu_link</child>
-      <parent>base_link</parent>
+      <child>$(arg vehicle_name)_plane/imu_link</child>
+      <parent>$(arg vehicle_name)_base_link</parent>
       <axis>
         <xyz>1 0 0</xyz>
@@ -95,5 +96,5 @@
       </axis>
     </joint>
-    <link name='rotor_puller'>
+    <link name='$(arg vehicle_name)_rotor_puller'>
       <pose>0.3 0 0.0 0 1.57 0</pose>
       <inertial>
@@ -109,5 +110,5 @@
         </inertia>
       </inertial>
-      <collision name='rotor_puller_collision'>
+      <collision name='$(arg vehicle_name)_rotor_puller_collision'>
         <pose>0.0 0 0.0 0 0 0</pose>
         <geometry>
@@ -126,5 +127,5 @@
         </surface>
       </collision>
-      <visual name='rotor_puller_visual'>
+      <visual name='$(arg vehicle_name)_rotor_puller_visual'>
         <pose>0 0 -0.09 0 0 0</pose>
         <geometry>
@@ -145,7 +146,7 @@
       <self_collide>0</self_collide>
     </link>
-    <joint name='rotor_puller_joint' type='revolute'>
-      <child>rotor_puller</child>
-      <parent>base_link</parent>
+    <joint name='$(arg vehicle_name)_rotor_puller_joint' type='revolute'>
+      <child>$(arg vehicle_name)_rotor_puller</child>
+      <parent>$(arg vehicle_name)_base_link</parent>
       <axis>
         <xyz>1 0 0</xyz>
@@ -161,5 +162,5 @@
       </axis>
     </joint>
-    <link name="left_elevon">
+    <link name="$(arg vehicle_name)_left_elevon">
       <inertial>
         <mass>0.00000001</mass>
@@ -175,5 +176,5 @@
       </inertial>
     </link>
-    <link name="right_elevon">
+    <link name="$(arg vehicle_name)_right_elevon">
       <inertial>
         <mass>0.00000001</mass>
@@ -189,5 +190,5 @@
       </inertial>
     </link>
-    <link name="elevator">
+    <link name="$(arg vehicle_name)_elevator">
       <inertial>
         <mass>0.00000001</mass>
@@ -203,5 +204,5 @@
       </inertial>
     </link>
-    <link name="rudder">
+    <link name="$(arg vehicle_name)_rudder">
       <inertial>
         <mass>0.00000001</mass>
@@ -217,7 +218,7 @@
       </inertial>
     </link>
-    <joint name='left_elevon_joint' type='revolute'>
-      <parent>base_link</parent>
-      <child>left_elevon</child>
+    <joint name='$(arg vehicle_name)_left_elevon_joint' type='revolute'>
+      <parent>$(arg vehicle_name)_base_link</parent>
+      <child>$(arg vehicle_name)_left_elevon</child>
       <pose>0 0.3 0 0.00 0 0.0</pose>
       <axis>
@@ -238,7 +239,7 @@
       </physics>
     </joint>
-    <joint name='right_elevon_joint' type='revolute'>
-      <parent>base_link</parent>
-      <child>right_elevon</child>
+    <joint name='$(arg vehicle_name)_right_elevon_joint' type='revolute'>
+      <parent>$(arg vehicle_name)_base_link</parent>
+      <child>$(arg vehicle_name)_right_elevon</child>
       <pose>0 -0.3 0 0.00 0 0.0</pose>
       <axis>
@@ -259,7 +260,7 @@
       </physics>
     </joint>
-    <joint name='elevator_joint' type='revolute'>
-      <parent>base_link</parent>
-      <child>elevator</child>
+    <joint name='$(arg vehicle_name)_elevator_joint' type='revolute'>
+      <parent>$(arg vehicle_name)_base_link</parent>
+      <child>$(arg vehicle_name)_elevator</child>
       <pose> -0.5 0 0 0 0 0</pose>
       <axis>
@@ -280,7 +281,7 @@
       </physics>
     </joint>
-    <joint name='rudder_joint' type='revolute'>
-      <parent>base_link</parent>
-      <child>rudder</child>
+    <joint name='$(arg vehicle_name)_rudder_joint' type='revolute'>
+      <parent>$(arg vehicle_name)_base_link</parent>
+      <child>$(arg vehicle_name)_rudder</child>
       <pose>-0.5 0 0.05 0.00 0 0.0</pose>
       <axis>
@@ -315,7 +316,7 @@
       <forward>1 0 0</forward>
       <upward>0 0 1</upward>
-      <link_name>base_link</link_name>
+      <link_name>$(arg vehicle_name)_base_link</link_name>
       <control_joint_name>
-        left_elevon_joint
+        $(arg vehicle_name)_left_elevon_joint
       </control_joint_name>
       <control_joint_rad_to_cl>-0.5</control_joint_rad_to_cl>
@@ -335,11 +336,11 @@
       <forward>1 0 0</forward>
       <upward>0 0 1</upward>
-      <link_name>base_link</link_name>
+      <link_name>$(arg vehicle_name)_base_link</link_name>
       <control_joint_name>
-        right_elevon_joint
+        $(arg vehicle_name)_right_elevon_joint
       </control_joint_name>
       <control_joint_rad_to_cl>-0.5</control_joint_rad_to_cl>
     </plugin>
-    <plugin name="elevator" filename="libLiftDragPlugin.so">
+    <plugin name="$(arg vehicle_name)_elevator" filename="libLiftDragPlugin.so">
       <a0>-0.2</a0>
       <cla>4.752798721</cla>
@@ -355,11 +356,11 @@
       <forward>1 0 0</forward>
       <upward>0 0 1</upward>
-      <link_name>base_link</link_name>
+      <link_name>$(arg vehicle_name)_base_link</link_name>
       <control_joint_name>
-        elevator_joint
+        $(arg vehicle_name)_elevator_joint
       </control_joint_name>
       <control_joint_rad_to_cl>-4.0</control_joint_rad_to_cl>
     </plugin>
-    <plugin name="rudder" filename="libLiftDragPlugin.so">
+    <plugin name="$(arg vehicle_name)_rudder" filename="libLiftDragPlugin.so">
       <a0>0.0</a0>
       <cla>4.752798721</cla>
@@ -375,10 +376,10 @@
       <forward>1 0 0</forward>
       <upward>0 1 0</upward>
-      <link_name>base_link</link_name>
+      <link_name>$(arg vehicle_name)_base_link</link_name>
     </plugin>
     <plugin name='puller' filename='libgazebo_motor_model.so'>
       <robotNamespace></robotNamespace>
-      <jointName>rotor_puller_joint</jointName>
-      <linkName>rotor_puller</linkName>
+      <jointName>$(arg vehicle_name)_rotor_puller_joint</jointName>
+      <linkName>$(arg vehicle_name)_rotor_puller</linkName>
       <turningDirection>cw</turningDirection>
       <timeConstantUp>0.0125</timeConstantUp>
@@ -396,5 +397,5 @@
     <plugin name='gazebo_imu_plugin' filename='libgazebo_imu_plugin.so'>
       <robotNamespace></robotNamespace>
-      <linkName>plane/imu_link</linkName>
+      <linkName>$(arg vehicle_name)_plane/imu_link</linkName>
       <imuTopic>/imu</imuTopic>
       <gyroscopeNoiseDensity>0.0003394</gyroscopeNoiseDensity>
@@ -408,6 +409,6 @@
     </plugin>
     <plugin name='wind_plugin' filename='libgazebo_wind_plugin.so'>
-      <frameId>base_link</frameId>
-      <linkName>base_link</linkName>
+      <frameId>$(arg vehicle_name)_base_link</frameId>
+      <linkName>$(arg vehicle_name)_base_link</linkName>
       <robotNamespace/>
       <xyzOffset>1 0 0</xyzOffset>
@@ -463,7 +464,7 @@
           <zero_position_armed>0</zero_position_armed>
           <joint_control_type>velocity</joint_control_type>
-          <joint_name>rotor_puller_joint</joint_name>
+          <joint_name>$(arg vehicle_name)_rotor_puller_joint</joint_name>
         </channel>
-        <channel name="left_elevon">
+        <channel name="$(arg vehicle_name)_left_elevon">
           <input_index>5</input_index>
           <input_offset>0</input_offset>
@@ -472,7 +473,7 @@
           <zero_position_armed>0</zero_position_armed>
           <joint_control_type>position_kinematic</joint_control_type>
-          <joint_name>left_elevon_joint</joint_name>
+          <joint_name>$(arg vehicle_name)_left_elevon_joint</joint_name>
         </channel>
-        <channel name="right_elevon">
+        <channel name="$(arg vehicle_name)_right_elevon">
           <input_index>6</input_index>
           <input_offset>0</input_offset>
@@ -481,7 +482,7 @@
           <zero_position_armed>0</zero_position_armed>
           <joint_control_type>position_kinematic</joint_control_type>
-          <joint_name>right_elevon_joint</joint_name>
+          <joint_name>$(arg vehicle_name)_right_elevon_joint</joint_name>
         </channel>
-        <channel name="elevator">
+        <channel name="$(arg vehicle_name)_elevator">
           <input_index>7</input_index>
           <input_offset>0</input_offset>
@@ -490,14 +491,22 @@
           <zero_position_armed>0</zero_position_armed>
           <joint_control_type>position_kinematic</joint_control_type>
-          <joint_name>elevator_joint</joint_name>
+          <joint_name>$(arg vehicle_name)_elevator_joint</joint_name>
         </channel>
       </control_channels>
     </plugin>
     <static>0</static>
+    <plugin name="joint_state_publisher" filename="libgazebo_ros_joint_state_publisher.so">
+      <ros>
+        <namespace>/demo</namespace>
+        <argument>joint_states:=joint_states</argument>
+      </ros>
+      <joint_name>$(arg vehicle_name)::$(arg vehicle_name)_rotor_puller_joint</joint_name>
+      <update_rate>100</update_rate>
+    </plugin>
   <xacro:if value="$(arg enable_camera)">
     <xacro:include filename="$(arg rotors_description_dir)/geotagged_cam/geotagged_cam.sdf.xacro">
     </xacro:include>
     <joint name="geotagged_cam_joint" type="fixed">
-      <parent>base_link</parent>
+      <parent>$(arg vehicle_name)_base_link</parent>
       <child>geotagged_cam::camera_link</child>
     </joint>

Commit message: Adding all joint to joint_state_publisher

File: models/iris/iris.sdf.xacro (robot description, xacro)
@@ -76,5 +76,5 @@
       </inertial>
     </link>
-    <joint name='imu_joint' type='revolute'>
+    <joint name='$(arg vehicle_name)_imu_joint' type='revolute'>
       <child>$(arg vehicle_name)_imu_link</child>
       <parent>$(arg vehicle_name)_base_link</parent>
@@ -568,8 +568,5 @@
     </plugin>
     <plugin name="joint_state_publisher" filename="libgazebo_ros_joint_state_publisher.so">
-      <ros>
-        <namespace>/</namespace>
-        <argument>joint_states:=joint_states</argument>
-      </ros>
+        <joint_name>$(arg vehicle_name)::$(arg vehicle_name)_imu_joint</joint_name>
       <joint_name>$(arg vehicle_name)::$(arg vehicle_name)_rotor_0_joint</joint_name>
       <joint_name>$(arg vehicle_name)::$(arg vehicle_name)_rotor_1_joint</joint_name>

File: models/iris/iris.urdf.xacro (robot description, xacro)
@@ -45,5 +45,5 @@
       </inertial>
     </link>
-    <joint name="imu_joint" type="revolute">
+    <joint name='$(arg vehicle_name)_imu_joint' type='revolute'>
       <parent link="$(arg vehicle_name)_base_link"/>
       <child link="$(arg vehicle_name)_imu_link"/>
@@ -408,9 +408,5 @@
     <static>0</static>
     <plugin name="joint_state_publisher" filename="libgazebo_ros_joint_state_publisher.so">
-      <ros>
-        <namespace>/</namespace>
-        <argument>joint_states:=joint_states</argument>
-      </ros>
-      <joint_name>$(arg vehicle_name)::$(arg vehicle_name)_imu_link</joint_name>
+      <joint_name>$(arg vehicle_name)::$(arg vehicle_name)_imu_joint</joint_name>
       <joint_name>$(arg vehicle_name)::$(arg vehicle_name)_rotor_0_joint</joint_name>
       <joint_name>$(arg vehicle_name)::$(arg vehicle_name)_rotor_1_joint</joint_name>

Commit message: added argument to allow ir_camera

File: models/iris/iris.sdf.xacro (robot description, xacro)
@@ -4,4 +4,5 @@
   <xacro:arg name='qgc_udp_port' default='4560' />
   <xacro:arg name='enable_camera' default='true' />
+  <xacro:arg name='enable_ir_camera' default='true' />
   <xacro:arg name='camera_pose' default='0 0 0 0 0 0' />
   <xacro:arg name='camera_udp_port' default='5600' />
@@ -604,4 +605,12 @@
     </joint>
   </xacro:if>
-  </model>
+  <xacro:if value="$(arg enable_ir_camera)">
+    <xacro:include filename="$(arg rotors_description_dir)/ir_cam/ir_cam.sdf.xacro">
+    </xacro:include>
+    <joint name="ir_camera_joint" type="fixed">
+      <parent>$(arg vehicle_name)_base_link</parent>
+      <child>ir_camera_link</child>
+    </joint>
+  </xacro:if>
+ </model>
 </sdf>
