Commit message: Fix plane mesh path

File: models/plane/plane.urdf.xacro (robot description, xacro)
@@ -23,5 +23,5 @@
         <origin rpy="0  0  0" xyz="0.07 0 0.166"/>
         <geometry>
-          <mesh filename="package://mavlink_sitl_gazebo/models/plane/meshes/body.dae" scale="0.1 0.1 0.1"/>
+          <mesh filename="package://plane/meshes/body.dae" scale="0.1 0.1 0.1"/>
         </geometry>
         <material name="Gazebo/DarkGrey">
@@ -67,5 +67,5 @@
         <origin rpy="0  0  0" xyz="0 0 -0.09"/>
         <geometry>
-          <mesh filename="package://mavlink_sitl_gazebo/models/plane/meshes/iris_prop_ccw.dae" scale="1 1 1"/>
+          <mesh filename="package://plane/meshes/iris_prop_ccw.dae" scale="1 1 1"/>
         </geometry>
         <material name="Gazebo/Blue">
